File: Arduino/untitled.brd (EAGLE design)
At the start: 100 x 80 mm, 142 parts, among them J3 USB-MICRO!!!, J4 3x2M, J5 HEAD17-NOSS, J6 HEAD17-NOSS-1, K1001 RT174005, K1101 RT174005, K1201 RT174005, K1401 RT174005, Q1001 BSS138L, Q1101 BSS138L, Q1201 BSS138L, Q1401 BSS138L, T1 FDN340P/PMV48XP, T2 PMV48XP, U1 LM2594M-12, U2 LM2594M-05, U3 ATMEGA32U4-XUMU, U4 LP2985-33DBVR, U5 NCP1117-5, Y3 16MHz KX-7

Commit message: schem look done
Parts:
- removed 0-10V1:C2: 0.1uF, rcl:C0603
- removed 0-10V1:R4: 100k, rcl:R0603
- removed C16, C17: 22pF, gen_comp:C0402
- removed C18, C19: 22u, rcl:SMC_B
- removed D+, D-: DNP, Arduino-utility:TP-1.00MM
- removed D1002, D1102, D1202, D1402: MBR0520LT, diode:SOD123
- removed F1: MF-MSMF050-2 500mA, rcl:L1812
- removed J3: USB-MICRO!!!, gen_comp:CON2_USB_MICRO_B_AT
- removed J5: HEAD17-NOSS, gen_comp:HEAD17-NOSS
- removed J6: HEAD17-NOSS-1, gen_comp:HEAD17-NOSS-1
- removed K1001, K1101, K1201, K1401: RT174005, relay:RT-C/O12A3.5
- removed L: green, led:CHIPLED_0805
- removed L3: MH2029-300Y, wuerth-elektronik:0805
- removed LED1001, LED1101, LED1201, LED1401, SENSE1:LED1, SENSE2:LED1, SENSE3:LED1, SENSE4:LED1: IN-S63AT5A, led:CHIP-LED0603
- removed ON: blue, led:CHIPLED_0805
- removed Q1001, Q1101, Q1201, Q1401: BSS138L, BSS138L:BSS138L
- removed R1001, R1101, R1201, R1401: 1K, eagle-ltspice:R0603
- removed R1002, R1102, R1202, R1402: 620, eagle-ltspice:R0603
- removed RESET: TS42, Arduino:TS42
- removed RX, TX: yellow, led:CHIPLED_0805
- removed SENSE1:B1, SENSE2:B1, SENSE3:B1, SENSE4:B1: B6S, rectifier:MBS
- removed SENSE1:OK1, SENSE2:OK1, SENSE3:OK1, SENSE4:OK1: LTV816S, optocoupler-3-jcn:SMD4
- removed SENSE1:R1, SENSE1:R2, SENSE2:R1, SENSE2:R2, SENSE3:R1, SENSE3:R2, SENSE4:R1, SENSE4:R2: 82K, rcl:R1206
- removed T2: PMV48XP, zetex:SOT-23
- removed U$37, U$53: DNP, Arduino-utility:FD-1-1.5
- removed U4: LP2985-33DBVR, gen_comp:SOT23-DBV
- removed U5: NCP1117-5, gen_comp:SOT223
- removed Y3: 16MHz KX-7, gen_comp:CRYSTAL-3.2-2.5
- removed Z1, Z2: CG0603MLC-05E, varistor:CT/CN0603
- added B501, B601, B701, B801: B6S, rectifier:MBS
- added D102, D202, D302, D402: MBR0520LT, diode:SOD123
- added D1101: CDSOT23-SM712, CDSOT23-SM712:SOT-23-3
- added IC1101: MAX481CSA, maxim:SO08
- added K101, K201, K301, K401: RT174005, relay:RT-C/O12A3.5
- added LED1, LED5, LED6: green, led:CHIPLED_0805
- added LED101, LED201, LED301, LED401, LED501, LED601, LED701, LED801: IN-S85AT5B, led:CHIP-LED0805
- added LED2, LED3: yellow, led:CHIPLED_0805
- added LED4: blue, led:CHIPLED_0805
- added OK501, OK601, OK701, OK801: LTV816S, optocoupler-3-jcn:SMD4
- added P1: KMMVX-SMT-BS-BTR, KMMVX-SMT-BS-BTR:KYCON_KMMVX-SMT-BS-BTR
- added Q101, Q201, Q301, Q401: BSS138L, BSS138L:BSS138L
- added R10: 600, rcl:R0603
- added R101, R201, R301, R401: 1K, eagle-ltspice:R0603
- added R102, R202, R302, R402: 300, eagle-ltspice:R0603
- added R3: 10K, rcl:R0402
- added R501, R502, R601, R602, R701, R702, R801, R802: 82K, rcl:R1206
- added S1: 430481035816_430481035816, 430481035816:430481035816
- added X13: (no value), con-wago-500:W237-103
- C1, C2: value 100uFx35V -> 22pF; device rcl:UD-6,3X7,7_NICHICON -> rcl:C0402
- C10, C12, C14: value 100n -> 100uFx35V; device gen_comp:C0402 -> rcl:UD-6,3X7,7_NICHICON
- C11: value 1uF -> 100uFx35V; device gen_comp:C0402 -> rcl:UD-6,3X7,7_NICHICON
- C13: value 1uF -> 100uFx6,3; device gen_comp:C0402 -> rcl:UD-6,3X5,8_NICHICON
- C15: value 100n -> 100uFx6,3; device gen_comp:C0402 -> rcl:UD-6,3X5,8_NICHICON
- C3, C5: value 100uFx35V -> 1uF; device rcl:UD-6,3X7,7_NICHICON -> rcl:C0402
- C4, C6: value 100uFx6,3 -> 100n; device rcl:UD-6,3X5,8_NICHICON -> rcl:C0402
- C7: device gen_comp:C0402 -> rcl:C0402
- C8: value 100n -> 22u; device gen_comp:C0402 -> rcl:SMC_B
- C9: value 1uF -> 100n; device gen_comp:C0402 -> rcl:C0402
- D1: value MBR0520LT -> CD1206-S01575; device diode:SOD123 -> diode:MINIMELF
- D2: value MBR0520LT -> MBRS130LT3; device diode:SOD123 -> diode:SMB
- D3: value CD1206-S01575 -> MBRS130LT3; device diode:MINIMELF -> diode:SMB
- L1, L2: value SRR0805-101K -> DO3316-224
- R1, R2: device gen_comp:R0402 -> rcl:R0402
- R4, R9: value 10K -> 600; device gen_comp:R0402 -> rcl:R0603
- R5: value 1K -> 600; device rcl:R0402 -> rcl:R0603
- R503, R603, R703, R803: value 620 -> 300
- R6, R7: value 1K -> 600; device gen_comp:R0402 -> rcl:R0603
- R8: value 1K -> 10K; device gen_comp:R0402 -> rcl:R0402
- U1: value LM2594M-12 -> MCU-ATMEGA32U4-MUR(VQFN44); device LM2594M-12:SOIC127P620X175-8N -> MCU-ATMEGA32U4-MUR_VQFN44_:QFN44G-0.5-7X7MM
- U2: value LM2594M-05 -> LM2594M-12
- U3: value ATMEGA32U4-XUMU -> LM2594M-05; device gen_comp:QFN44ML7X7 -> LM2594M-12:SOIC127P620X175-8N
- X1: value (none) -> 16MHz KX-7; device con-wago-500:W237-103 -> gen_comp:CRYSTAL-3.2-2.5
- moved U1 925.4 mm to (-212.1, -1115.1)
- moved D1 896.1 mm to (-1.70, -1118.7)
- moved C2 696.4 mm to (-0.65, -894.4)
- moved C1 672.9 mm to (-0.65, -881.7)
- moved R9 671.6 mm to (-214.6, 148.6)
- moved C5 665.2 mm to (-0.65, -932.5)
- moved C4 663.9 mm to (-0.65, -919.8)
- moved C3 662.7 mm to (-0.65, -907.1)
- moved X12 597.2 mm to (76.2, 78.7), turned to 180 degrees
- moved C6 580.7 mm to (-0.65, -856.3)
- moved X11 579.5 mm to (61.0, 78.7), turned to 180 degrees
- moved X10 560.1 mm to (40.6, 78.7), turned to 180 degrees
- moved R4 555.5 mm to (-0.85, -1046.8)
- moved X9 542.8 mm to (25.4, 78.7), turned to 180 degrees
- moved R6 526.9 mm to (-0.85, -1021.4)
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- renumbered 0-10V1:C1 to C901, 0-10V1:IC1 to IC901, 0-10V1:R1 to R901, 0-10V1:R2 to R902, 0-10V1:R3 to R903, 0-10V1:R5 to R905, 0-10V1:R6 to R906, J4 to JP1, RP3 to RN1, RS485-1:D1 to D1001, RS485-1:IC1 to IC1001, SENSE1:C1 to C501, SENSE1:R3 to R503, SENSE1:R4 to R504, SENSE1:R5 to R505, SENSE2:C1 to C601, SENSE2:R3 to R603, SENSE2:R4 to R604, SENSE2:R5 to R605, SENSE3:C1 to C701, SENSE3:R3 to R703, SENSE3:R4 to R704, SENSE3:R5 to R705, SENSE4:C1 to C801, SENSE4:R3 to R803, SENSE4:R4 to R804, SENSE4:R5 to R805
Connections:
- removed net +VIN: C12.1, T2.2, U5.3
- removed net 0-10V1:N$7: 0-10V1:C2.1, 0-10V1:R4.2, IC901.5
- removed net 0-10V1:N$8: IC901.6, R905.2, R906.1
- removed net 0-10V1:PWM_IN_1: R901.1
- removed net 0-10V1:PWM_IN_2: 0-10V1:R4.1
- removed net 10V2: IC901.7, R906.2, X11.3
- removed net 3V3: C9.1, J6.16, U4.5
- removed net A0: J6.14, U3.36
- removed net A1: J6.13, U3.37
- removed net A2: J6.12, U3.38
- removed net A3: J6.11, U3.39
- removed net AVCC: C13.1, L3.2, U3.44
- removed net D0/RX: J5.4, U3.20
- removed net D1/TX: J5.3, U3.21
- removed net D2/SDA: J5.7, U3.19
- removed net D3/SCL: J5.8, U3.18
- removed net D4*: J5.9, U3.25
- removed net D5*: J5.10, U3.31
- removed net D6*: J5.11, U3.27
- removed net D7: J5.12, U3.1
- removed net IO10*: J5.15, U3.30
- removed net IO11*: J5.16, U3.12
- removed net IO12*: J5.17, U3.26
- removed net IO13*: J6.17, R8.1, U3.32
- removed net IO8: J5.13, U3.28
- removed net IO9*: J5.14, U3.29
- removed net N$3: X10.1
- removed net N$7: X10.3
- removed net RELAY1:INPUT: R1001.1
- removed net RELAY2:INPUT: R1101.1
- removed net RELAY3:INPUT: R1201.1
- removed net RELAY4:INPUT: R1401.1
- removed net RS485-1:485D: IC1001.4
- removed net RS485-1:485R: IC1001.1
- removed net RS485-1:485REDE: IC1001.2, IC1001.3
- removed net RS485A: D1001.2, IC1001.7, X8.2
- removed net RS485B: D1001.1, IC1001.6, X8.1
- removed net SENSE1:OUTPUT: R505.2
- removed net SENSE2:OUTPUT: R605.2
- removed net SENSE3:OUTPUT: R705.2
- removed net SENSE4:OUTPUT: R805.2
- removed net VIN: J6.3, R9.2, T1.3, T2.1
- removed net VUSBD: C18.+, F1.1, J3.P1
- new net 0-10V1:N$1: IC901.5, R905.1, R906.2
- new net 0-10V1:N$3: IC901.6, IC901.7
- new net A0/S1: R505.2, U1.36
- new net A1/S2: R605.2, U1.37
- new net A2/S3: R705.2, U1.38
- new net A3/S4: R805.2, U1.39
- new net A4O: RN1.6, X10.2
- new net A5O: RN1.5, X11.2
- new net D0/RX/RS485R2: IC1101.1, U1.20
- new net D1/TX/RS485D2: IC1101.4, U1.21
- new net D2/SDA/RS485REDE2: IC1101.2, IC1101.3, U1.19
- new net D3/SCL/PWM: R901.1, U1.18
- new net D4/R1: R101.1, U1.25
- new net D5/R2: R201.1, U1.31
- new net D6/R3: R301.1, U1.27
- new net D7/R4: R401.1, U1.1
- new net IO10/RS485REDE1: IC1001.2, IC1001.3, U1.30
- new net IO11: R10.1, U1.12, X4.3
- new net IO12: R9.1, U1.26, X12.1
- new net IO13: R4.1, U1.32
- new net IO8/RS485R1: IC1001.1, U1.28
- new net IO9/RS485D1: IC1001.4, U1.29
- new net N$10: R2.2, T1.3
- new net N$16: LED5.A, R9.2
- new net N$17: LED6.A, R10.2
- new net RS485A1: D1001.2, IC1001.7, X9.1
- new net RS485A2: D1101.2, IC1101.7, X9.3
- new net RS485B1: D1001.1, IC1001.6, X8.3
- new net RS485B2: D1101.1, IC1101.6, X9.2
- net +12V: now also C12.+, C14.+, R905.2, U2.4; no longer C3.+, C5.+, U1.4
- net +5V: now also C13.+, C15.+, C3.1, C6.1, C7.1, D1.C, D102.C, D202.C, D302.C, D402.C, IC1101.8, K101.A2, K201.A2, K301.A2, K401.A2, OK501.4, OK601.4, OK701.4, OK801.4, R102.2, R202.2, R302.2, R402.2, R7.1, U1.14, U1.2, U1.24, U1.34, U1.44, U3.4, X10.1, X11.1; no longer C14.1, C15.1, C19.+, C4.+, C6.+, C8.1, D1002.C, D1102.C, D1202.C, D1402.C, D3.C, J6.6, K1001.A2, K1101.A2, K1201.A2, K1401.A2, L3.1, R1002.2, R1102.2, R1202.2, R1402.2, R5.1, SENSE1:OK1.4, SENSE2:OK1.4, SENSE3:OK1.4, SENSE4:OK1.4, T2.3, U2.4, U3.14, U3.2, U3.24, U3.34, U4.1, U4.3, U5.2, U5.4
- net 10V1: now also X12.2; no longer X11.1
- net 24V1: now also X8.1; no longer X7.1
- net 24V2: now also X8.2; no longer X7.2
- net A4: now also RN1.3, U1.40; no longer J6.10, U3.40
- net A5: now also RN1.4, U1.41; no longer J6.9, U3.41
- net AREF: now also C4.1, U1.42; no longer C7.1, J6.15, U3.42
- net D+: now also P1.3; no longer D+.X, J3.P3, Z1.1
- net D-: now also P1.2; no longer D-.X, J3.P2, Z2.1
- net GND: now also C1.1, C10.-, C11.-, C12.-, C13.-, C14.-, C15.-, C2.1, C3.2, C4.2, C5.2, C6.2, C8.-, D1101.3, D3.A, IC1101.5, LED1.C, LED2.C, LED3.C, LED4.C, LED5.C, LED501.C, LED6.C, LED601.C, LED701.C, LED801.C, P1.5, Q101.S, Q201.S, Q301.S, Q401.S, R3.1, R8.2, R906.1, S1.3, S1.4, U1.15, U1.23, U1.35, U1.43, U1.TAB, U3.6, X1.2, X1.4, X10.3, X11.3, X12.3; no longer 0-10V1:C2.2, C1.-, C10.2, C11.2, C12.2, C13.2, C14.2, C15.2, C16.1, C17.1, C18.-, C19.-, C2.-, C3.-, C4.-, C5.-, C6.-, C8.2, D1.A, J3.P5, J3.S1, J3.S2, J3.S3, J3.S4, J3.S5, J3.S6, J5.6, J6.4, L.C, ON.C, Q1001.S, Q1101.S, Q1201.S, Q1401.S, R4.2, R9.1, R905.1, RESET.3, RESET.4, RESET.5, RN1.3, RN1.4, RN1.5, RN1.6, RX.C, SENSE1:LED1.C, SENSE2:LED1.C, SENSE3:LED1.C, SENSE4:LED1.C, TX.C, U1.6, U3.15, U3.23, U3.35, U3.43, U3.EXP, U4.2, U5.1, X11.2, X7.3, X8.3, Y3.2, Y3.4, Z1.2, Z2.2
- net HWB: now also R8.1, U1.33; no longer R4.1, U3.33
- net MISO: now also U1.11; no longer J6.2, U3.11
- net MOSI: now also U1.10; no longer J5.1, U3.10
- net N$1: now also C10.+, C11.+, U3.7; no longer C1.+, C2.+, U1.7
- net N$2: now also D2.C, U2.8; no longer D1.C, U1.8
- net N$4: now also LED1.A, R4.2; no longer L.A, R8.2
- net N$5: now also LED2.A, R5.2; no longer R7.2, RX.A
- net N$6: now also LED3.A; no longer TX.A
- net N$8: now also D3.C, U3.8; no longer D2.C, U2.8
- net N$9: now also LED4.A, R7.2; no longer ON.A, R5.2
- net R1G: now also K101.11, X5.1; no longer K1001.11, X4.1
- net R1NC: now also K101.12, X5.2; no longer K1001.12, X4.2
- net R1NO: now also K101.14, X5.3; no longer K1001.14, X4.3
- net R2G: now also K201.11, X6.1; no longer K1101.11, X5.1
- net R2NC: now also K201.12, X6.2; no longer K1101.12, X5.2
- net R2NO: now also K201.14, X6.3; no longer K1101.14, X5.3
- net R3G: now also K301.11, X7.1; no longer K1201.11, X6.1
- net R3NC: now also K301.12, X7.2; no longer K1201.12, X6.2
- net R3NO: now also K301.14, X7.3; no longer K1201.14, X6.3
- net R4G: now also K401.11, X13.3; no longer K1401.11, X12.3
- net R4NC: now also K401.12, X13.2; no longer K1401.12, X12.2
- net R4NO: now also K401.14, X13.1; no longer K1401.14, X12.1
- net RD+: now also U1.4; no longer U3.4
- net RD-: now also U1.3; no longer U3.3
- net RELAY1:N$1: now also D102.A, K101.A1, LED101.C, Q101.D; no longer D1002.A, K1001.A1, LED1001.C, Q1001.D
- net RELAY1:N$2: now also LED101.A, R102.1; no longer LED1001.A, R1002.1
- net RELAY1:N$4: now also Q101.G, R101.2; no longer Q1001.G, R1001.2
- net RELAY2:N$1: now also D202.A, K201.A1, LED201.C, Q201.D; no longer D1102.A, K1101.A1, LED1101.C, Q1101.D
- net RELAY2:N$2: now also LED201.A, R202.1; no longer LED1101.A, R1102.1
- net RELAY2:N$4: now also Q201.G, R201.2; no longer Q1101.G, R1101.2
- net RELAY3:N$1: now also D302.A, K301.A1, LED301.C, Q301.D; no longer D1202.A, K1201.A1, LED1201.C, Q1201.D
- net RELAY3:N$2: now also LED301.A, R302.1; no longer LED1201.A, R1202.1
- net RELAY3:N$4: now also Q301.G, R301.2; no longer Q1201.G, R1201.2
- net RELAY4:N$1: now also D402.A, K401.A1, LED401.C, Q401.D; no longer D1402.A, K1401.A1, LED1401.C, Q1401.D
- net RELAY4:N$2: now also LED401.A, R402.1; no longer LED1401.A, R1402.1
- net RELAY4:N$4: now also Q401.G, R401.2; no longer Q1401.G, R1401.2
- net RESET: now also D1.A, S1.1, S1.2, U1.13; no longer D3.A, J5.5, J6.5, RESET.1, RESET.2, U3.13
- net RXLED/SS: now also R5.1, U1.8; no longer J5.2, R7.1, U3.8
- net S11: now also B501.AC1, X2.2; no longer SENSE1:B1.AC1, X1.1
- net S12: now also B501.AC2, X2.1; no longer SENSE1:B1.AC2, X1.2
- net S21: now also B601.AC1, X3.1; no longer SENSE2:B1.AC1, X1.3
- net S22: now also B601.AC2, X2.3; no longer SENSE2:B1.AC2, X2.1
- net S31: now also B701.AC1, X3.3; no longer SENSE3:B1.AC1, X2.2
- net S32: now also B701.AC2, X3.2; no longer SENSE3:B1.AC2, X2.3
- net S41: now also B801.AC1, X4.2; no longer SENSE4:B1.AC1, X3.1
- net S42: now also B801.AC2, X4.1; no longer SENSE4:B1.AC2, X3.2
- net SCK: now also U1.9; no longer J6.1, U3.9
- net SENSE1:N$10: now also OK501.3; no longer SENSE1:OK1.3
- net SENSE1:N$2: now also LED501.A; no longer SENSE1:LED1.A
- net SENSE1:N$3: now also B501.+, R501.1; no longer SENSE1:B1.+, SENSE1:R1.1
- net SENSE1:N$4: now also OK501.1, R501.2; no longer SENSE1:OK1.1, SENSE1:R1.2
- net SENSE1:N$5: now also OK501.2, R502.2; no longer SENSE1:OK1.2, SENSE1:R2.2
- net SENSE1:N$6: now also B501.-, R502.1; no longer SENSE1:B1.-, SENSE1:R2.1
- net SENSE2:N$10: now also OK601.3; no longer SENSE2:OK1.3
- net SENSE2:N$2: now also LED601.A; no longer SENSE2:LED1.A
- net SENSE2:N$3: now also B601.+, R601.1; no longer SENSE2:B1.+, SENSE2:R1.1
- net SENSE2:N$4: now also OK601.1, R601.2; no longer SENSE2:OK1.1, SENSE2:R1.2
- net SENSE2:N$5: now also OK601.2, R602.2; no longer SENSE2:OK1.2, SENSE2:R2.2
- net SENSE2:N$6: now also B601.-, R602.1; no longer SENSE2:B1.-, SENSE2:R2.1
- net SENSE3:N$10: now also OK701.3; no longer SENSE3:OK1.3
- net SENSE3:N$2: now also LED701.A; no longer SENSE3:LED1.A
- net SENSE3:N$3: now also B701.+, R701.1; no longer SENSE3:B1.+, SENSE3:R1.1
- net SENSE3:N$4: now also OK701.1, R701.2; no longer SENSE3:OK1.1, SENSE3:R1.2
- net SENSE3:N$5: now also OK701.2, R702.2; no longer SENSE3:OK1.2, SENSE3:R2.2
- net SENSE3:N$6: now also B701.-, R702.1; no longer SENSE3:B1.-, SENSE3:R2.1
- net SENSE4:N$10: now also OK801.3; no longer SENSE4:OK1.3
- net SENSE4:N$2: now also LED801.A; no longer SENSE4:LED1.A
- net SENSE4:N$3: now also B801.+, R801.1; no longer SENSE4:B1.+, SENSE4:R1.1
- net SENSE4:N$4: now also OK801.1, R801.2; no longer SENSE4:OK1.1, SENSE4:R1.2
- net SENSE4:N$5: now also OK801.2, R802.2; no longer SENSE4:OK1.2, SENSE4:R2.2
- net SENSE4:N$6: now also B801.-, R802.1; no longer SENSE4:B1.-, SENSE4:R2.1
- net TXLED: now also U1.22; no longer U3.22
- net UCAP: now also C5.1, U1.6; no longer C11.1, U3.6
- net VUSB: now also C8.+, C9.1, P1.1, R3.2, U1.7; no longer C10.1, F1.2, R2.2, U3.7
- net XTAL1: now also C2.2, U1.17, X1.3; no longer C17.2, U3.17, Y3.3
- net XTAL2: now also C1.2, U1.16, X1.1; no longer C16.2, U3.16, Y3.1
Other:
- board size 100 x 80 mm -> 101.5 x 86.3 mm

Commit message: first try:
Parts:
- removed C13, C15: 100uFx6,3, rcl:UD-6,3X5,8_NICHICON
- removed C14: 100uFx35V, rcl:UD-6,3X7,7_NICHICON
- removed R505, R605, R705, R805: 10k, rcl:R0603
- C10, C11: value 100uFx35V -> 220uFx35V; device rcl:UD-6,3X7,7_NICHICON -> rcl:UD-10X10_NICHICON
- C12: value 100uFx35V -> 220uFx10; device rcl:UD-6,3X7,7_NICHICON -> rcl:UD-6,3X5,8_NICHICON
- L1: value DO3316-224 -> DO3308P-334MLD
- LED1, LED5, LED6: value green -> IN-S85AT5B; device led:CHIPLED_0805 -> led:CHIP-LED0805
- LED2, LED3: value yellow -> IN-S85AT5B; device led:CHIPLED_0805 -> led:CHIP-LED0805
- LED4: value blue -> IN-S85AT5B; device led:CHIPLED_0805 -> led:CHIP-LED0805
- R10, R9: value 600 -> 10K; device rcl:R0603 -> rcl:R0402
- R102, R202, R302, R402, R503, R603, R703, R803: value 300 -> 600; device eagle-ltspice:R0603 -> rcl:R0603
- R3, R8: value 10K -> 600; device rcl:R0402 -> rcl:R0603
- R504, R604, R704, R804: value 10 -> 10K; device rcl:R0603 -> rcl:R0402
- R901: value 100k -> 10k; device rcl:R0603 -> rcl:R0402
- R902, R903, R905, R906: device rcl:R0603 -> rcl:R0402
- moved P1 1216.6 mm to (49.5, 63.5)
- moved IC1101 1210.2 mm to (27.3, 71.8), turned to 90 degrees
- moved D1101 1208.3 mm to (21.0, 69.8), turned to 90 degrees
- moved U1 1185.1 mm to (47.6, 41.3)
- moved S1 1184.8 mm to (35.6, 63.5), turned to 180 degrees
- moved LED4 1183.6 mm to (48.9, 77.7), turned to 90 degrees
- moved D1 1181.5 mm to (28.8, 62.4), turned to 270 degrees
- moved LED3 1170.9 mm to (48.9, 79.8), turned to 90 degrees
- moved LED2 1158.2 mm to (48.9, 81.9), turned to 90 degrees
- moved LED1 1145.5 mm to (48.9, 84.0), turned to 90 degrees
- moved R4 1116.2 mm to (57.1, 67.9)
- moved R5 1107.2 mm to (60.7, 71.4)
- moved R6 1090.8 mm to (61.4, 67.6)
- moved R7 1082.2 mm to (65.2, 71.4)
- moved R8 1065.7 mm to (65.8, 67.6)
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Connections:
- removed net SENSE1:N$9: C501.+, R504.1
- removed net SENSE2:N$9: C601.+, R604.1
- removed net SENSE3:N$9: C701.+, R704.1
- removed net SENSE4:N$9: C801.+, R804.1
- net +12V: now also C11.+; no longer C12.+, C14.+
- net +5V: now also C12.+, R8.1; no longer C13.+, C15.+, R7.1
- net 24V1: now also X8.3; no longer X8.1
- net A0/S1: now also R504.2; no longer R505.2
- net A1/S2: now also R604.2; no longer R605.2
- net A2/S3: now also R704.2; no longer R705.2
- net A3/S4: now also R804.2; no longer R805.2
- net GND: now also R10.1, R9.2; no longer C13.-, C14.-, C15.-, R3.1, R8.2
- net HWB: now also R9.1; no longer R8.1
- net IO11: now also R3.1; no longer R10.1
- net IO12: now also R4.1; no longer R9.1
- net IO13: now also R5.1; no longer R4.1
- net N$1: no longer C11.+
- net N$10: now also R10.2; no longer R2.2
- net N$16: now also LED2.A, R4.2; no longer LED5.A, R9.2
- net N$17: now also LED1.A, R3.2; no longer LED6.A, R10.2
- net N$4: now also LED3.A, R5.2; no longer LED1.A, R4.2
- net N$5: now also LED4.A, R6.2; no longer LED2.A, R5.2
- net N$6: now also LED5.A, R7.2; no longer LED3.A, R6.2
- net N$9: now also LED6.A, R8.2; no longer LED4.A, R7.2
- net R1G: now also X5.3; no longer X5.1
- net R1NO: now also X5.1; no longer X5.3
- net R2G: now also X6.3; no longer X6.1
- net R2NO: now also X6.1; no longer X6.3
- net R3G: now also X7.3; no longer X7.1
- net R3NO: now also X7.1; no longer X7.3
- net RS485A1: now also X9.3; no longer X9.1
- net RS485A2: now also X9.1; no longer X9.3
- net RS485B1: now also X8.1; no longer X8.3
- net RXLED/SS: now also R6.1; no longer R5.1
- net SENSE1:N$10: now also C501.+, R504.1; no longer R504.2, R505.1
- net SENSE2:N$10: now also C601.+, R604.1; no longer R604.2, R605.1
- net SENSE3:N$10: now also C701.+, R704.1; no longer R704.2, R705.1
- net SENSE4:N$10: now also C801.+, R804.1; no longer R804.2, R805.1
- net TXLED: now also R7.1; no longer R6.1
- net VUSB: now also R2.2; no longer R3.2
Routing:
- net GND: track 0.00 -> 519.4 mm, vias 0 -> 12
- net +5V: track 0.00 -> 360.7 mm, vias 0 -> 12
- net +12V: track 0.00 -> 87.0 mm, vias 0 -> 2
- net RELAY4:N$1: track 0.00 -> 79.3 mm
- net IO11: track 0.00 -> 76.7 mm, vias 0 -> 2
- net SENSE1:N$2: track 0.00 -> 70.2 mm, vias 0 -> 2
- net D3/SCL/PWM: track 0.00 -> 64.7 mm
- net IO10/RS485REDE1: track 0.00 -> 55.6 mm, vias 0 -> 2
- net D7/R4: track 0.00 -> 54.7 mm, vias 0 -> 2
- net SENSE2:N$2: track 0.00 -> 54.4 mm, vias 0 -> 2
- net SENSE3:N$2: track 0.00 -> 51.7 mm, vias 0 -> 2
- net D6/R3: track 0.00 -> 51.1 mm
- net RELAY1:N$1: track 0.00 -> 48.4 mm, vias 0 -> 2
- net RD-: track 0.00 -> 46.6 mm
- net MOSI: track 0.00 -> 44.1 mm
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