File: Arduino/untitled.sch (EAGLE design)
At the start: 71 parts, among them J3 USB-MICRO!!!, J4 3x2M, J5 HEAD17-NOSS, J6 HEAD17-NOSS-1, T1 FDN340P/PMV48XP, T2 PMV48XP, U1 LM2594M-12, U2 LM2594M-05, U3 ATMEGA32U4-XUMU, U4 LP2985-33DBVR, U5 NCP1117-5, Y3 16MHz KX-7

Commit message: schem look done
Parts:
- removed C16, C17: 22pF, gen_comp:C-EUC0402
- removed C18, C19: 22u, rcl:CPOL-EUSMCB
- removed D+, D-: DNP, Arduino-utility:TPTP-1.00MM
- removed F1: MF-MSMF050-2 500mA, rcl:L-EUL1812
- removed J3: USB-MICRO!!!, gen_comp:MYCON2_USB-MINI-B
- removed J4: 3x2M, gen_comp:PINHD-2X3
- removed J5: HEAD17-NOSS, gen_comp:HEAD17-NOSS
- removed J6: HEAD17-NOSS-1, gen_comp:HEAD17-NOSS-1
- removed L: green, led:LEDCHIPLED_0805
- removed L3: MH2029-300Y, wuerth-elektronik:WE-CBF_0805
- removed ON: blue, led:LEDCHIPLED_0805
- removed RESET: TS42, Arduino:TS42
- removed RP3: 22R, resistor-dil:4R-NCAY16
- removed RX, TX: yellow, led:LEDCHIPLED_0805
- removed T2: PMV48XP, zetex:PMOSSOT23
- removed U$37, U$53: DNP, Arduino-utility:FIDUCIAL-1.5MM
- removed U4: LP2985-33DBVR, gen_comp:LP2985-XXDBVR33
- removed U5: NCP1117-5, gen_comp:LINEAR_MC33269ST
- removed Y3: 16MHz KX-7, gen_comp:CRYSTAL-3.2-2.5
- removed Z1, Z2: CG0603MLC-05E, varistor:VARISTORCN0603
- added JP1: 3x2M, gen_comp:PINHD-2X3
- added LED1, LED5, LED6: green, led:LEDCHIPLED_0805
- added LED2, LED3: yellow, led:LEDCHIPLED_0805
- added LED4: blue, led:LEDCHIPLED_0805
- added P1: KMMVX-SMT-BS-BTR, KMMVX-SMT-BS-BTR:KMMVX-SMT-BS-BTR
- added R10: 600, rcl:R-EU_R0603
- added R3: 10K, rcl:R-EU_R0402
- added RN1: 22R, resistor-dil:4R-NCAY16
- added S1: 430481035816_430481035816, 430481035816:430481035816_430481035816
- added X13: (no value), con-wago-500:W237-103
- C1, C2: value 100uFx35V -> 22pF; device rcl:CPOL-EUUD-6,3X7,7 -> rcl:C-EUC0402; MODEL UWT1V101MCL1GS -> (none)
- C10, C12, C14: value 100n -> 100uFx35V; device gen_comp:C-EUC0402 -> rcl:CPOL-EUUD-6,3X7,7; MODEL (none) -> UWT1V101MCL1GS
- C11: value 1uF -> 100uFx35V; device gen_comp:C-EUC0402 -> rcl:CPOL-EUUD-6,3X7,7; MODEL (none) -> UWT1V101MCL1GS
- C13: value 1uF -> 100uFx6,3; device gen_comp:C-EUC0402 -> rcl:CPOL-EUUD-6,3X8,8
- C15: value 100n -> 100uFx6,3; device gen_comp:C-EUC0402 -> rcl:CPOL-EUUD-6,3X8,8
- C3, C5: value 100uFx35V -> 1uF; device rcl:CPOL-EUUD-6,3X7,7 -> rcl:C-EUC0402; MODEL UWT1V101MCL1GS -> (none)
- C4, C6: value 100uFx6,3 -> 100n; device rcl:CPOL-EUUD-6,3X8,8 -> rcl:C-EUC0402
- C7: device gen_comp:C-EUC0402 -> rcl:C-EUC0402
- C8: value 100n -> 22u; device gen_comp:C-EUC0402 -> rcl:CPOL-EUSMCB
- C9: value 1uF -> 100n; device gen_comp:C-EUC0402 -> rcl:C-EUC0402
- D1: value MBR0520LT -> CD1206-S01575; device diode:MBR0520LT -> diode:DIODE-MINIMELF
- D2: value MBR0520LT -> MBRS130LT3; device diode:MBR0520LT -> diode:MBRS130LT3
- D3: value CD1206-S01575 -> MBRS130LT3; device diode:DIODE-MINIMELF -> diode:MBRS130LT3
- L1, L2: value SRR0805-101K -> DO3316-224
- R1, R2: device gen_comp:R-EU_R0402 -> rcl:R-EU_R0402
- R4, R9: value 10K -> 600; device gen_comp:R-EU_R0402 -> rcl:R-EU_R0603
- R5: value 1K -> 600; device rcl:R-EU_R0402 -> rcl:R-EU_R0603
- R6, R7: value 1K -> 600; device gen_comp:R-EU_R0402 -> rcl:R-EU_R0603
- R8: value 1K -> 10K; device gen_comp:R-EU_R0402 -> rcl:R-EU_R0402
- U1: value LM2594M-12 -> MCU-ATMEGA32U4-MUR(VQFN44); device LM2594M-12:LM2594M-12 -> MCU-ATMEGA32U4-MUR_VQFN44_:MCU-ATMEGA32U4-MUR(VQFN44)
- U2: value LM2594M-05 -> LM2594M-12
- U3: value ATMEGA32U4-XUMU -> LM2594M-05; device gen_comp:ATMEGA32U4-XUMU -> LM2594M-12:LM2594M-12
- X1: value (none) -> 16MHz KX-7; device con-wago-500:W237-103 -> gen_comp:CRYSTAL-3.2-2.5
Connections:
- removed net +VIN: C12.1, T2.S, U5.IN
- removed net 0-10V_2: R6.2
- removed net 10V2: X11-3.KL
- removed net 3V3: C9.1, J6.16, U4.OUT
- removed net A0: J6.14, U3.(ADC7/TDI)PF7
- removed net A1: J6.13, U3.(ADC6/TDO)PF6
- removed net A2: J6.12, U3.(ADC5/TMS)PF5
- removed net A3: J6.11, U3.(ADC4/TCK)PF4
- removed net AVCC: C13.1, L3.2, U3.AVCC1
- removed net D0/RX: J5.4, U3.(RXD1/AIN1/INT2)PD2
- removed net D1/TX: J5.3, U3.(TXD1/INT3)PD3
- removed net D2/SDA: J5.7, U3.(SDA/INT1)PD1
- removed net D3/SCL: J5.8, U3.(OC0B/SCL/INT0)PD0
- removed net D4*: J5.9, U3.(ICP1/ADC8)PD4
- removed net D5*: J5.10, U3.(OC3A/#0C4A)PC6
- removed net D6*: J5.11, U3.(T0/OC4D/ADC10)PD7
- removed net D7: J5.12, U3.(INT6/AIN0)PE6
- removed net IO10*: J5.15, U3.(PCINT6/OC1B/OC4B/ADC13)PB6
- removed net IO11*: J5.16, U3.(PCINT7/OC0A/OC1C/#RTS)PB7
- removed net IO12*: J5.17, U3.(T1/#OC4D/ADC9)PD6
- removed net IO13*: J6.17, R8.1, U3.(ICP3/CLK0/OC4A)PC7
- removed net IO8: J5.13, U3.(ADC11/PCINT4)PB4
- removed net IO9*: J5.14, U3.(PCINT5/OC1A/#OC4B/ADC12)PB5
- removed net N$7: C2.1, R4.2, X10-3.KL
- removed net PWM_IN_2: R4.1
- removed net VIN: J6.3, R9.2, T1.G, T2.D
- removed net VUSBD: C18.+, F1.1, J3.VBUS
- new net 0-10V_1: R3.2
- new net A0/S1: U1.PF7(ADC7/TDI)
- new net A1/S2: U1.PF6(ADC6/TDO)
- new net A2/S3: U1.PF5(ADC5/TMS)
- new net A3/S4: U1.PF4(ADC4/TCK)
- new net A4O: RN1C.2, X10-2.KL
- new net A5O: RN1D.2, X11-2.KL
- new net D0/RX/RS485R2: U1.PD2(RXD1/INT2)
- new net D1/TX/RS485D2: U1.PD3(TXD1/INT3)
- new net D2/SDA/RS485REDE2: U1.PD1(SDA/INT1)
- new net D3/SCL/PWM: U1.PD0(OC0B/SCL/INT0)
- new net D4/R1: U1.PD4(ICP1/ADC8)
- new net D5/R2: U1.PC6(OC3A/!OC4A)
- new net D6/R3: U1.PD7(T0/OC4D/ADC10)
- new net D7/R4: U1.PE6(INT.6/AIN0)
- new net IO10/RS485REDE1: U1.PB6(PCINT6/OC1B/OC4B/ADC13)
- new net IO11: R10.1, U1.PB7(PCINT7/OC0A/OC1C/!RTS), X4-3.KL
- new net IO12: R9.1, U1.PD6(T1/ADC9/!OC4D), X12-1.KL
- new net IO13: R4.1, U1.PC7(ICP3/CLK0/OC4A)
- new net IO8/RS485R1: U1.PB4(PCINT4/ADC11)
- new net IO9/RS485D1: U1.PB5(PCINT5/OC1A/ADC12/!OC4B)
- new net N$16: LED5.A, R9.2
- new net N$17: LED6.A, R10.2
- new net RS485A1: X9-1.KL
- new net RS485A2: X9-3.KL
- new net RS485B1: X8-3.KL
- new net RS485B2: X9-2.KL
- net +12V: now also C12.+, C14.+, R5.2, U2.FB; no longer C3.+, C5.+, U1.FB
- net +5V: now also C13.+, C15.+, C3.1, C6.1, C7.1, D1.C, JP1.2, R7.1, U1.AVCC@1, U1.AVCC@2, U1.UVCC, U1.VCC@1, U1.VCC@2, U3.FB, X10-1.KL, X11-1.KL; no longer C14.1, C15.1, C19.+, C4.+, C6.+, C8.1, D3.C, J4.2, J6.6, L3.1, R5.1, T2.G, U2.FB, U3.AVCC, U3.UVCC, U3.VCC, U3.VCC1, U4.IN, U4.ON/!OFF, U5.OUT, U5.OUT@1
- net 10V1: now also X12-2.KL; no longer X11-1.KL
- net 24V1: now also X8-1.KL; no longer X7-1.KL
- net 24V2: now also X8-2.KL; no longer X7-2.KL
- net A4: now also RN1C.1, U1.PF1(ADC1); no longer J6.10, U3.(ADC1)PF1
- net A5: now also RN1D.1, U1.PF0(ADC0); no longer J6.9, U3.(ADC0)PF0
- net AREF: now also C4.1, U1.AREF; no longer C7.1, J6.15, U3.AREF
- net D+: now also P1.D+, RN1A.2; no longer D+.P$1, J3.D+, RP3A.2, Z1.1
- net D-: now also P1.D-, RN1B.2; no longer D-.P$1, J3.D-, RP3B.2, Z2.1
- net GND: now also C1.1, C10.-, C11.-, C12.-, C13.-, C14.-, C15.-, C2.1, C3.2, C4.2, C5.2, C6.2, C8.-, D3.A, JP1.6, LED1.C, LED2.C, LED3.C, LED4.C, LED5.C, LED6.C, P1.GND, R3.1, R6.1, R8.2, S1.3, S1.4, U1.GND@1, U1.GND@2, U1.GND@3, U1.GND@4, U1.UGND, U3.~ON~/OFF, X1.GND@1, X1.GND@2, X10-3.KL, X11-3.KL, X12-3.KL; no longer C10.2, C11.2, C12.2, C13.2, C14.2, C15.2, C16.1, C17.1, C18.-, C19.-, C2.-, C2.2, C3.-, C4.-, C5.-, C6.-, C8.2, D1.A, J3.GND, J3.SH1, J3.SH2, J3.SH3, J3.SH4, J3.SH5, J3.SH6, J4.6, J5.6, J6.4, L.C, ON.C, R4.2, R5.1, R9.1, RESET.3, RESET.4, RESET.5-GND, RP3C.1, RP3C.2, RP3D.1, RP3D.2, RX.C, TX.C, U1.GND, U1.~ON~/OFF, U3.GND1, U3.GND2, U3.GND3, U3.PAD, U3.UGND, U4.GND, U5.GND/ADJ, X11-2.KL, X7-3.KL, X8-3.KL, Y3.GND@1, Y3.GND@2, Z1.2, Z2.2
- net HWB: now also R8.1, U1.PE2(!HWB); no longer R4.1, U3.(#HWB)PE2
- net MISO: now also JP1.1, U1.PB3(PD0/PCINT3/MISO); no longer J4.1, J6.2, U3.(PD0/MISO/PCINT3)PB3
- net MOSI: now also JP1.4, U1.PB2(PDI/PCINT2/MOSI); no longer J4.4, J5.1, U3.(PDI/MOSI/PCINT2)PB2
- net N$1: now also C10.+, C11.+, LED1.C, R5.1, R6.2, U3.VIN; no longer C1.+, C2.+, U1.VIN
- net N$10: now also R2.2, R3.2, T1.G
- net N$2: now also D2.C, LED1.A, R3.1, U2.OUT; no longer D1.C, U1.OUT
- net N$3: no longer X10-1.KL
- net N$4: now also LED1.A, R3.1, R4.2; no longer L.A, R8.2
- net N$5: now also LED2.A, R5.2; no longer R7.2, RX.A
- net N$6: now also LED3.A; no longer TX.A
- net N$8: now also D3.C, U3.OUT; no longer D2.C, R5.2, R6.1, U2.OUT
- net N$9: now also LED4.A, R7.2; no longer ON.A, R5.2
- net R1G: now also X5-1.KL; no longer X4-1.KL
- net R1NC: now also X5-2.KL; no longer X4-2.KL
- net R1NO: now also X5-3.KL; no longer X4-3.KL
- net R2G: now also X6-1.KL; no longer X5-1.KL
- net R2NC: now also X6-2.KL; no longer X5-2.KL
- net R2NO: now also X6-3.KL; no longer X5-3.KL
- net R3G: now also X7-1.KL; no longer X6-1.KL
- net R3NC: now also X7-2.KL; no longer X6-2.KL
- net R3NO: now also X7-3.KL; no longer X6-3.KL
- net R4G: now also X13-3.KL; no longer X12-3.KL
- net R4NC: now also X13-2.KL; no longer X12-2.KL
- net R4NO: now also X13-1.KL; no longer X12-1.KL
- net RD+: now also RN1A.1, U1.D+; no longer RP3A.1, U3.D+
- net RD-: now also RN1B.1, U1.D-; no longer RP3B.1, U3.D-
- net RESET: now also D1.A, JP1.5, S1.1, S1.2, U1.!RESET; no longer D3.A, J4.5, J5.5, J6.5, RESET.1, RESET.2, U3.RESET
- net RS485A: no longer X8-2.KL
- net RS485B: no longer X8-1.KL
- net RXLED/SS: now also R5.1, U1.PB0(SS/PCINT0); no longer J5.2, R7.1, U3.(SS/PCINT0)PB0
- net S11: now also X2-2.KL; no longer X1-1.KL
- net S12: now also X2-1.KL; no longer X1-2.KL
- net S21: now also X3-1.KL; no longer X1-3.KL
- net S22: now also X2-3.KL; no longer X2-1.KL
- net S31: now also X3-3.KL; no longer X2-2.KL
- net S32: now also X3-2.KL; no longer X2-3.KL
- net S41: now also X4-2.KL; no longer X3-1.KL
- net S42: now also X4-1.KL; no longer X3-2.KL
- net SCK: now also JP1.3, U1.PB1(PCINT1/SCLK); no longer J4.3, J6.1, U3.(SCLK/PCINT1)PB1
- net TXLED: now also U1.PD5(XCLK1/!CTS); no longer U3.(XCK1/#CTS)PD5
- net UCAP: now also C5.1, U1.UCAP; no longer C11.1, U3.UCAP
- net VUSB: now also C8.+, C9.1, P1.VCC, R3.2, U1.VBUS; no longer C10.1, F1.2, R2.2, U3.VBUS
- net XTAL1: now also C2.2, U1.XTAL1, X1.C2; no longer C17.2, U3.XTAL1, Y3.C2
- net XTAL2: now also C1.2, U1.XTAL2, X1.C1; no longer C16.2, U3.XTAL2, Y3.C1
Other:
- note removed: "#PWM 10bit"
- note removed: "#PWM 16bit"
- note removed: "#PWM 8/16bit"
- note removed: "#PWM 8bit"
- note removed: "#PWM Hi-Speed"
- note removed: "+3V3 REG"
- note removed: "+5V REG"
- note removed: "NOT USED"
- note removed: "USB"

Commit message: first try:
Parts:
- removed C13, C15: 100uFx6,3, rcl:CPOL-EUUD-6,3X8,8
- removed C14: 100uFx35V, rcl:CPOL-EUUD-6,3X7,7
- C10, C11: value 100uFx35V -> 220uFx35V; device rcl:CPOL-EUUD-6,3X7,7 -> rcl:CPOL-EUUD-10X10
- C12: value 100uFx35V -> 220uFx10; device rcl:CPOL-EUUD-6,3X7,7 -> rcl:CPOL-EUUD-6,3X8,8; MODEL UWT1V101MCL1GS -> (none)
- L1: value DO3316-224 -> DO3308P-334MLD
- LED1, LED5, LED6: value green -> IN-S85AT5B; device led:LEDCHIPLED_0805 -> led:LEDCHIP-LED0805
- LED2, LED3: value yellow -> IN-S85AT5B; device led:LEDCHIPLED_0805 -> led:LEDCHIP-LED0805
- LED4: value blue -> IN-S85AT5B; device led:LEDCHIPLED_0805 -> led:LEDCHIP-LED0805
- R10, R9: value 600 -> 10K; device rcl:R-EU_R0603 -> rcl:R-EU_R0402
- R3, R8: value 10K -> 600; device rcl:R-EU_R0402 -> rcl:R-EU_R0603
Connections:
- net +12V: now also C11.+; no longer C12.+, C14.+
- net +5V: now also C12.+, R8.1; no longer C13.+, C15.+, R7.1
- net 24V1: now also X8-3.KL; no longer X8-1.KL
- net GND: now also R10.1, R9.2; no longer C13.-, C14.-, C15.-, R3.1, R8.2
- net HWB: now also R9.1; no longer R8.1
- net IO11: now also R3.1; no longer R10.1
- net IO12: now also R4.1; no longer R9.1
- net IO13: now also R5.1; no longer R4.1
- net N$1: no longer C11.+
- net N$10: now also C1.+, R10.2, R4.1; no longer R2.2, R4.2, R5.1
- net N$16: now also LED2.A, R4.2; no longer LED5.A, R9.2
- net N$17: now also LED1.A, R3.2; no longer LED6.A, R10.2
- net N$4: now also LED3.A, R5.2; no longer LED1.A, R4.2
- net N$5: now also LED4.A, R6.2; no longer LED2.A, R5.2
- net N$6: now also LED5.A, R7.2; no longer LED3.A, R6.2
- net N$9: now also LED6.A, R8.2; no longer C1.+, LED4.A, R4.1, R7.2
- net OUTPUT: now also R4.2; no longer R5.2
- net R1G: now also X5-3.KL; no longer X5-1.KL
- net R1NO: now also X5-1.KL; no longer X5-3.KL
- net R2G: now also X6-3.KL; no longer X6-1.KL
- net R2NO: now also X6-1.KL; no longer X6-3.KL
- net R3G: now also X7-3.KL; no longer X7-1.KL
- net R3NO: now also X7-1.KL; no longer X7-3.KL
- net RS485A1: now also X9-3.KL; no longer X9-1.KL
- net RS485A2: now also X9-1.KL; no longer X9-3.KL
- net RS485B1: now also X8-1.KL; no longer X8-3.KL
- net RXLED/SS: now also R6.1; no longer R5.1
- net TXLED: now also R7.1; no longer R6.1
- net VUSB: now also R2.2; no longer R3.2
Other:
- moved on the sheet: C11, C12, LED1, LED2, LED3, LED4, LED5, LED6, R10, R2, R3, R4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
